Commit message: Complete SLAM mapping and save map

File: src/serving_robot_description/urdf/serving_robot.urdf (robot description, URDF)
Before this commit: robot serving_robot, 21 links, 20 joints
Joints:
- joint caster_wheel_joint: type continuous -> fixed

Commit message: Add restaurant world and fix SLAM/Gazebo configuration

File: src/serving_robot_description/urdf/serving_robot.urdf (robot description, URDF)
Before this commit: robot serving_robot, 21 links, 20 joints
Joints:
- joint left_wheel_joint: origin xyz=0.03 0.14 -0.04 rpy=0 0 0 -> xyz=0.06 0.14 -0.04 rpy=0 0 0
- joint right_wheel_joint: origin xyz=0.03 -0.14 -0.04 rpy=0 0 0 -> xyz=0.06 -0.14 -0.04 rpy=0 0 0
